File: hv-downconverter/hv-downconverter.kicad_sch (KiCad schematic)
At the start: 13 parts, among them J1 Conn_01x02_Pin, U1 LM5116MHX/NOPB

Commit message: schematic captured, starting to place components
Parts:
- added C7: 1u, Capacitor_SMD:C_0805_2012Metric, symbol Device:C_Small
- added C8: 100n, Capacitor_SMD:C_0805_2012Metric, symbol Device:C_Small
- added C9: 22u, Capacitor_SMD:C_1210_3225Metric, symbol Device:C_Small
- added D1: BAS516, Diode_SMD:D_SOD-523, symbol Diode:BAS516
- added J2: Conn_01x02_Pin, Connector_PinHeader_2.54mm:PinHeader_1x02_P2.54mm_Vertical, symbol Connector:Conn_01x02_Pin
- added L1: 1.2u, Inductor_SMD:L_Coilcraft_XAL7070-XXX, symbol Device:L_Small
- added Q1, Q2: Q_NMOS_GDS, Package_TO_SOT_SMD:PQFN_8x8, symbol Device:Q_NMOS_GDS
- added R6: 3m, Resistor_SMD:R_1206_3216Metric, symbol Device:R_Small_US
- added R7: 62k, Resistor_SMD:R_0805_2012Metric, symbol Device:R_Small_US
- added R8: 11.1k, Resistor_SMD:R_0805_2012Metric, symbol Device:R_Small_US
- C1: footprint (none) -> Capacitor_SMD:C_1210_3225Metric
- C2, C3, C4, C5, C6: footprint (none) -> Capacitor_SMD:C_0805_2012Metric
- J1: footprint (none) -> Connector_PinHeader_2.54mm:PinHeader_1x02_P2.54mm_Vertical
- R1, R2, R3, R4, R5: footprint (none) -> Resistor_SMD:R_0805_2012Metric
Connections:
- net at C1.1, C2.1, J1.1 (Pin_1)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: now also Q1.2 (D)
- net at U1.10 (VOUT): now also C9.1, J2.1 (Pin_1), L1.2, R7.1
- net GND: now reaches U1.11 (DEMB)
- net GND: now also C1.2, C2.2, C3.2, C4.2, J1.2 (Pin_2), R2.2, R3.2, U1.13 (CSG), U1.14 (PGND), U1.17 (VCCX), U1.6 (AGND), C7.2, C9.2, J2.2 (Pin_2), R6.2, R8.2
- net at U1.12 (CS): now also Q2.3 (S), R6.1
- net at U1.15 (LO): now also Q2.1 (G)
- net at U1.16 (VCC): now also C7.1, D1.2 (A)
- net at U1.18 (HB): now also C8.1, D1.1 (K)
- net at U1.19 (HO): now also Q1.1 (G)
- net at U1.20 (SW): now also C8.2, L1.1, Q1.3 (S), Q2.2 (D)
- net at C5.2, C6.2, U1.8 (FB): now also R7.2, R8.1
Other:
- moved on the sheet: C1, C2, C3, C4, C5, C6, J1, R1, R2, R3, R4, R5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

Commit message: almost ready for fab
Parts:
- removed Q1, Q2: Q_NMOS_GDS, Package_TO_SOT_SMD:PQFN_8x8, symbol Device:Q_NMOS_GDS
- added Q3, Q4: Q_NMOS_GSD, Package_TO_SOT_SMD:PQFN_8x8, symbol Device:Q_NMOS_GSD
- C2, C3, C4, C5, C6, C8: footprint Capacitor_SMD:C_0805_2012Metric -> Capacitor_SMD:C_0603_1608Metric
- C9: footprint Capacitor_SMD:C_1210_3225Metric -> Capacitor_SMD:C_2220_5650Metric
- R2, R3, R4, R5, R7, R8: footprint Resistor_SMD:R_0805_2012Metric -> Resistor_SMD:R_0603_1608Metric
Connections:
- net GND: now also U1.21 (DAP)
- net at U1.15 (LO): now also Q4.1 (G)
- net at C8.2, L1.1, U1.20 (SW): now also Q3.2 (S), Q4.3 (D)
- net at R6.1, U1.12 (CS): now also Q4.2 (S)
- net at C1.1, C2.1, J1.1 (Pin_1)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: now also Q3.3 (D)
- net at U1.19 (HO): now also Q3.1 (G)

Commit message: nearly at production
Parts:
- added C10, C11, C12: 1u, Capacitor_SMD:C_2220_5750Metric, symbol Device:C_Small
- C1: value 2.2u -> 1u; footprint Capacitor_SMD:C_1210_3225Metric -> Capacitor_SMD:C_2220_5750Metric
- C2: footprint Capacitor_SMD:C_0603_1608Metric -> Capacitor_SMD:C_0805_2012Metric
Connections:
- net GND: now also C10.2, C11.2, C12.2
- net at C1.1, C2.1, J1.1 (Pin_1)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: now also C10.1, C11.1, C12.1
Other:
- moved on the sheet: C1, C2, C3, C4, C5, C6, C7, C8, C9, D1, J1, J2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
