File: hvhf-downconverter/hvhf-downconverter.kicad_pcb (KiCad board)
At the start: 4 copper layers, 27 x 42.2 mm, 27 parts, among them J3 Conn_01x01_Pin, J5 Conn_01x01_Pin, Q3 Q_NMOS_GSD, Q4 Q_NMOS_GSD, U1 LM5116MHX/NOPB

Commit message: nearly at production
Parts:
- renumbered Vin to J1, Vout to J4
Routing:
- net Net-(J1-Pin_1): track 42.4 -> 45.0 mm
Other:
- board text removed: "DroneTether Buck v1 jomg 9.16.24"
Changed lines of the file:
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@@
 		(sheetname "Root")
 		(sheetfile "hv-downconverter.kicad_sch")
-		(attr smd exclude_from_pos_files exclude_from_bom)
+		(attr smd exclude_from_pos_files)
 		(fp_line
 			(start 4.11 -4.11)
@@
 		(sheetname "Root")
 		(sheetfile "hv-downconverter.kicad_sch")
-		(attr smd exclude_from_pos_files exclude_from_bom)
+		(attr smd exclude_from_pos_files)
 		(fp_line
 			(start 4.11 4.11)
@@
 		(sheetname "Root")
 		(sheetfile "hv-downconverter.kicad_sch")
-		(attr smd exclude_from_pos_files exclude_from_bom)
+		(attr smd exclude_from_pos_files)
 		(fp_line
 			(start -4.11 4.26)
@@
 		(sheetname "Root")
 		(sheetfile "hv-downconverter.kicad_sch")
-		(attr smd exclude_from_pos_files exclude_from_bom)
+		(attr smd exclude_from_pos_files)
 		(fp_line
 			(start -0.727064 0.91)
@@
 		(descr "Through hole straight pin header, 1x01, 2.54mm pitch, single row")
 		(tags "Through hole pin header THT 1x01 2.54mm single row")
-		(property "Reference" "Vin"
+		(property "Reference" "J1"
 			(at 0 -2.33 180)
 			(layer "F.SilkS")
@@
 			(at 0 -2.33 0)
 			(layer "F.SilkS")
-			(hide yes)
 			(effects
 				(font
@@
 		(tags "capacitor")
 		(property "Reference" "C10"
-			(at -5.5 0 0)
+			(at -5.5 0 360)
 			(layer "F.SilkS")
 			(effects
@@
 		)
 		(property "Value" "1u"
-			(at 0 3.65 0)
+			(at 0 3.65 360)
 			(layer "F.Fab")
 			(effects
@@
 		)
 		(fp_text user "${REFERENCE}"
-			(at 0 0 0)
+			(at 0 0 360)
 			(layer "F.Fab")
 			(effects
@@
 		(descr "Through hole straight pin header, 1x01, 2.54mm pitch, single row")
 		(tags "Through hole pin header THT 1x01 2.54mm single row")
-		(property "Reference" "Vout"
-			(at 3 0 0)
+		(property "Reference" "J4"
+			(at 0 -2.33 0)
 			(layer "F.SilkS")
 			(effects
@@
 		(sheetname "Root")
 		(sheetfile "hv-downconverter.kicad_sch")
-		(attr smd exclude_from_pos_files exclude_from_bom)
+		(attr smd exclude_from_pos_files)
 		(fp_line
 			(start -0.237258 -0.5225)
@@
 		)
 	)
-	(gr_line
-		(start 186 98.8)
-		(end 188 98.8)
-		(stroke
-			(width 0.15)
-			(type default)
-		)
-		(layer "F.SilkS")
-	)
-	(gr_line
-		(start 188 98.75)
-		(end 188 98.5)
-		(stroke
-			(width 0.15)
-			(type default)
-		)
-		(layer "F.SilkS")
-	)
-	(gr_line
-		(start 188 98.5)
-		(end 188 98)
-		(stroke
-			(width 0.15)
-			(type default)
-		)
-		(layer "F.SilkS")
-	)
-	(gr_line
-		(start 188 99.5)
-		(end 188 100)
-		(stroke
-			(width 0.15)
-			(type default)
-		)
-		(layer "F.SilkS")
-	)
-	(gr_line
-		(start 186 99.5)
-		(end 186 100)
-		(stroke
-			(width 0.15)
-			(type default)
-		)
-		(layer "F.SilkS")
-	)
-	(gr_line
-		(start 186 99.5)
-		(end 186 99.25)
-		(stroke
-			(width 0.15)
-			(type default)
-		)
-		(layer "F.SilkS")
-	)
-	(gr_line
-		(start 186 98.5)
-		(end 186 98.75)
-		(stroke
-			(width 0.15)
-			(type default)
-		)
-		(layer "F.SilkS")
-	)
 	(gr_circle
 		(center 174.5 67.5)
@@
 		(layer "F.SilkS")
 	)
-	(gr_line
-		(start 186 99.2)
-		(end 188 99.2)
-		(stroke
-			(width 0.15)
-			(type default)
-		)
-		(layer "F.SilkS")
-	)
-	(gr_line
-		(start 186 98)
-		(end 186 98.5)
-		(stroke
-			(width 0.15)
-			(type default)
-		)
-		(layer "F.SilkS")
-	)
-	(gr_line
-		(start 188 99.25)
-		(end 188 99.5)
-		(stroke
-			(width 0.15)
-			(type default)
-		)
-		(layer "F.SilkS")
-	)
-	(gr_circle
-		(center 187 99)
-		(end 188 100.5)
-		(stroke
-			(width 0.15)
-			(type default)
-		)
-		(fill none)
-		(layer "F.SilkS")
-	)
 	(gr_rect
 		(start 162.5 65.25)
@@
 		(layer "Edge.Cuts")
 	)
-	(gr_text "DroneTether Buck v1\njomg 9.16.24"
-		(at 163 91.7 270)
-		(layer "F.SilkS")
-		(effects
-			(font
-				(size 1 1)
-				(thickness 0.15)
-			)
-			(justify left bottom)
-		)
-	)
 	(segment
 		(start 171.001679 67.650499)
@@
 	)
 	(segment
+		(start 172.55 90.5)
+		(end 169.965 90.5)
+		(width 0.8)
+		(layer "F.Cu")
+		(net 1)
+	)
+	(segment
 		(start 167.1625 66.75)
 		(end 168.8375 66.75)
@@
 		(polygon
 			(pts
-				(xy 171 84.75) (xy 171 89.5) (xy 173 89.5) (xy 173 91.5) (xy 171 91.5) (xy 171 107.75) (xy 162.75 107.75)
-				(xy 162.75 84.75)
+				(xy 171 84.75) (xy 171 107.75) (xy 162.75 107.75) (xy 162.75 84.75)
 			)
 		)
@@
 			)
 		)
-	)
-	(zone
-		(net 0)
-		(net_name "")
-		(layer "F.Mask")
-		(hatch edge 0.5)
-		(connect_pads
-			(clearance 0.5)
-		)
-		(min_thickness 0.25)
-		(filled_areas_thickness no)
-		(fill yes
-			(thermal_gap 0.5)
-			(thermal_bridge_width 0.5)
-		)
-		(polygon
-			(pts
-				(xy 177.5 96) (xy 179.5 96) (xy 179.5 106.5) (xy 177.5 106.5)
-			)
-		)
-	)
-	(zone
-		(net 0)
-		(net_name "")
-		(layer "F.Mask")
-		(hatch edge 0.5)
-		(connect_pads
-			(clearance 0.5)
-		)
-		(min_thickness 0.25)
-		(filled_areas_thickness no)
-		(fill yes
-			(thermal_gap 0.5)
-			(thermal_bridge_width 0.5)
-		)
-		(polygon
-			(pts
-				(xy 185 107) (xy 181.5 107) (xy 181.5 96) (xy 185 96)
-			)
-		)
